File: Motor CC/MotorCC.brd (EAGLE design)
At the start: 47 x 58.1 mm, 11 parts

Commit message: Add the routes now !
Parts:
- moved C2 2.84 mm to (35.6, 12.7)
Routing:
- added copper zone on layer 1, net GND
Changed lines of the file:
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@@
 <elements>
 <element name="U$1" library="SparkFun-PowerIC" package="POWERSO20" value="L298_BRIDGE_DRIVER" x="17.78" y="11.43"/>
-<element name="C1" library="resistor" package="C0805" value="100nF" x="19.05" y="49.53"/>
-<element name="C2" library="resistor" package="C0805" value="100nF" x="33.02" y="11.43" rot="R90"/>
-<element name="D11" library="diode" package="SMA-DO214AC" value="GF1" x="27.94" y="46.99"/>
-<element name="D12" library="diode" package="SMA-DO214AC" value="GF1" x="27.94" y="39.37"/>
-<element name="D13" library="diode" package="SMA-DO214AC" value="GF1" x="27.94" y="31.75"/>
-<element name="D14" library="diode" package="SMA-DO214AC" value="GF1" x="27.94" y="24.13"/>
-<element name="D21" library="diode" package="SMA-DO214AC" value="GF1" x="8.89" y="46.99"/>
-<element name="D22" library="diode" package="SMA-DO214AC" value="GF1" x="8.89" y="39.37"/>
-<element name="D23" library="diode" package="SMA-DO214AC" value="GF1" x="8.89" y="31.75"/>
-<element name="D24" library="diode" package="SMA-DO214AC" value="GF1" x="8.89" y="24.13"/>
+<element name="C1" library="resistor" package="C0805" value="100nF" x="19.05" y="49.53" smashed="yes">
+<attribute name="NAME" x="18.161" y="50.546" size="1.27" layer="25"/>
+</element>
+<element name="C2" library="resistor" package="C0805" value="100nF" x="35.56" y="12.7" smashed="yes" rot="R90">
+<attribute name="NAME" x="34.544" y="11.811" size="1.27" layer="25" rot="R90"/>
+</element>
+<element name="D11" library="diode" package="SMA-DO214AC" value="GF1" x="27.94" y="46.99" smashed="yes">
+<attribute name="NAME" x="24.765" y="48.5775" size="1.27" layer="25"/>
+</element>
+<element name="D12" library="diode" package="SMA-DO214AC" value="GF1" x="27.94" y="39.37" smashed="yes">
+<attribute name="NAME" x="24.765" y="40.9575" size="1.27" layer="25"/>
+</element>
+<element name="D13" library="diode" package="SMA-DO214AC" value="GF1" x="27.94" y="31.75" smashed="yes">
+<attribute name="NAME" x="24.765" y="33.3375" size="1.27" layer="25"/>
+</element>
+<element name="D14" library="diode" package="SMA-DO214AC" value="GF1" x="27.94" y="24.13" smashed="yes">
+<attribute name="NAME" x="24.765" y="25.7175" size="1.27" layer="25"/>
+</element>
+<element name="D21" library="diode" package="SMA-DO214AC" value="GF1" x="8.89" y="46.99" smashed="yes">
+<attribute name="NAME" x="5.715" y="48.5775" size="1.27" layer="25"/>
+</element>
+<element name="D22" library="diode" package="SMA-DO214AC" value="GF1" x="8.89" y="39.37" smashed="yes">
+<attribute name="NAME" x="5.715" y="40.9575" size="1.27" layer="25"/>
+</element>
+<element name="D23" library="diode" package="SMA-DO214AC" value="GF1" x="8.89" y="31.75" smashed="yes">
+<attribute name="NAME" x="5.715" y="33.3375" size="1.27" layer="25"/>
+</element>
+<element name="D24" library="diode" package="SMA-DO214AC" value="GF1" x="8.89" y="24.13" smashed="yes">
+<attribute name="NAME" x="5.715" y="25.7175" size="1.27" layer="25"/>
+</element>
 </elements>
 <signals>
@@
 <contactref element="U$1" pad="20"/>
 <contactref element="C2" pad="2"/>
-<wire x1="6.84" y1="46.99" x2="19.9" y2="49.53" width="0" layer="19" extent="1-1"/>
-<wire x1="6.84" y1="39.37" x2="6.84" y2="46.99" width="0" layer="19" extent="1-1"/>
-<wire x1="6.84" y1="31.75" x2="6.84" y2="39.37" width="0" layer="19" extent="1-1"/>
-<wire x1="6.84" y1="24.13" x2="6.84" y2="31.75" width="0" layer="19" extent="1-1"/>
-<wire x1="11.049" y1="17.145" x2="6.84" y2="24.13" width="0" layer="19" extent="1-1"/>
-<wire x1="11.049" y1="5.715" x2="11.049" y2="17.145" width="0" layer="19" extent="1-1"/>
-<wire x1="24.511" y1="17.145" x2="11.049" y2="17.145" width="0" layer="19" extent="1-1"/>
-<wire x1="33.02" y1="12.28" x2="24.511" y2="17.145" width="0" layer="19" extent="1-1"/>
-<wire x1="24.511" y1="5.715" x2="33.02" y2="12.28" width="0" layer="19" extent="1-1"/>
+<polygon width="0.4064" layer="1">
+<vertex x="-3.81" y="0"/>
+<vertex x="-3.81" y="60.96"/>
+<vertex x="49.53" y="60.96"/>
+<vertex x="49.53" y="59.69"/>
+<vertex x="49.53" y="-3.81"/>
+<vertex x="-3.81" y="-3.81"/>
+</polygon>
 </signal>
 <signal name="N$1">
@@
 <contactref element="U$1" pad="12"/>
 <contactref element="C2" pad="1"/>
-<wire x1="24.511" y1="6.985" x2="33.02" y2="10.58" width="0" layer="19" extent="1-1"/>
+<wire x1="24.511" y1="6.985" x2="35.56" y2="11.85" width="0" layer="19" extent="1-1"/>
 </signal>
 <signal name="VSS">

Commit message: Routes added
Connections:
- net GND: no longer U$1.1, U$1.10, U$1.11, U$1.20
Routing:
- net VSS: track 0.00 -> 70.5 mm, vias 0 -> 2
- net N$1: track 0.00 -> 53.1 mm, vias 0 -> 2
- net N$2: track 0.00 -> 47.9 mm, vias 0 -> 2
- net N$3: track 0.00 -> 38.1 mm
- net N$4: track 0.00 -> 28.1 mm
- net VCC: track 0.00 -> 13.3 mm
Changed lines of the file:
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@@
 </variantdefs>
 <classes>
-<class number="0" name="default" width="0" drill="0">
+<class number="0" name="default" width="0.381" drill="0.508">
+<clearance class="0" value="0.508"/>
 </class>
 </classes>
@@
 <autorouter>
 <pass name="Default">
-<param name="RoutingGrid" value="50mil"/>
+<param name="RoutingGrid" value="10mil"/>
 <param name="tpViaShape" value="round"/>
 <param name="PrefDir.1" value="|"/>
@@
 <signals>
 <signal name="GND">
-<contactref element="U$1" pad="11"/>
-<contactref element="U$1" pad="10"/>
 <contactref element="C1" pad="2"/>
 <contactref element="D21" pad="A"/>
@@
 <contactref element="D24" pad="A"/>
 <contactref element="D23" pad="A"/>
-<contactref element="U$1" pad="1"/>
-<contactref element="U$1" pad="20"/>
 <contactref element="C2" pad="2"/>
 <polygon width="0.4064" layer="1">
-<vertex x="-3.81" y="0"/>
-<vertex x="-3.81" y="60.96"/>
-<vertex x="49.53" y="60.96"/>
-<vertex x="49.53" y="59.69"/>
-<vertex x="49.53" y="-3.81"/>
-<vertex x="-3.81" y="-3.81"/>
+<vertex x="-1.27" y="59.69"/>
+<vertex x="48.26" y="59.69"/>
+<vertex x="48.26" y="58.42"/>
+<vertex x="48.26" y="-1.27"/>
+<vertex x="-1.27" y="-1.27"/>
 </polygon>
 </signal>
@@
 <contactref element="D11" pad="A"/>
 <contactref element="D21" pad="K"/>
-<wire x1="10.94" y1="46.99" x2="25.89" y2="46.99" width="0" layer="19" extent="1-1"/>
-<wire x1="11.049" y1="13.335" x2="10.94" y2="46.99" width="0" layer="19" extent="1-1"/>
+<wire x1="25.89" y1="46.99" x2="19.304" y2="46.99" width="0.381" layer="1"/>
+<wire x1="19.304" y1="46.99" x2="10.94" y2="46.99" width="0.381" layer="1"/>
+<wire x1="12.954" y1="13.462" x2="11.176" y2="13.462" width="0.381" layer="1"/>
+<wire x1="19.304" y1="19.812" x2="12.954" y2="13.462" width="0.381" layer="16"/>
+<wire x1="19.304" y1="46.99" x2="19.304" y2="19.812" width="0.381" layer="16"/>
+<wire x1="11.176" y1="13.462" x2="11.049" y2="13.335" width="0.381" layer="1"/>
+<via x="12.954" y="13.462" extent="1-16" drill="0.6096"/>
+<via x="19.304" y="46.99" extent="1-16" drill="0.6096"/>
 </signal>
 <signal name="N$2">
@@
 <contactref element="D12" pad="A"/>
 <contactref element="D22" pad="K"/>
-<wire x1="10.94" y1="39.37" x2="25.89" y2="39.37" width="0" layer="19" extent="1-1"/>
-<wire x1="11.049" y1="12.065" x2="10.94" y2="39.37" width="0" layer="19" extent="1-1"/>
+<wire x1="25.89" y1="39.37" x2="12.954" y2="39.37" width="0.381" layer="1"/>
+<wire x1="12.954" y1="39.37" x2="10.94" y2="39.37" width="0.381" layer="1"/>
+<wire x1="9.144" y1="12.192" x2="10.922" y2="12.192" width="0.381" layer="1"/>
+<wire x1="9.144" y1="39.37" x2="9.144" y2="12.192" width="0.381" layer="16"/>
+<wire x1="12.954" y1="39.37" x2="9.144" y2="39.37" width="0.381" layer="16"/>
+<wire x1="10.922" y1="12.192" x2="11.049" y2="12.065" width="0.381" layer="1"/>
+<via x="9.144" y="12.192" extent="1-16" drill="0.6096"/>
+<via x="12.954" y="39.37" extent="1-16" drill="0.6096"/>
 </signal>
 <signal name="N$3">
@@
 <contactref element="D13" pad="A"/>
 <contactref element="D23" pad="K"/>
-<wire x1="10.94" y1="31.75" x2="25.89" y2="31.75" width="0" layer="19" extent="1-1"/>
-<wire x1="24.511" y1="12.065" x2="25.89" y2="31.75" width="0" layer="19" extent="1-1"/>
+<wire x1="25.89" y1="31.75" x2="10.94" y2="31.75" width="0.381" layer="1"/>
+<wire x1="27.432" y1="12.192" x2="24.638" y2="12.192" width="0.381" layer="1"/>
+<wire x1="27.432" y1="25.4" x2="27.432" y2="12.192" width="0.381" layer="1"/>
+<wire x1="25.908" y1="26.924" x2="27.432" y2="25.4" width="0.381" layer="1"/>
+<wire x1="25.908" y1="31.75" x2="25.908" y2="26.924" width="0.381" layer="1"/>
+<wire x1="24.638" y1="12.192" x2="24.511" y2="12.065" width="0.381" layer="1"/>
+<wire x1="25.908" y1="31.75" x2="25.89" y2="31.75" width="0.381" layer="1"/>
 </signal>
 <signal name="N$4">
@@
 <contactref element="D14" pad="A"/>
 <contactref element="D24" pad="K"/>
-<wire x1="24.511" y1="13.335" x2="25.89" y2="24.13" width="0" layer="19" extent="1-1"/>
-<wire x1="10.94" y1="24.13" x2="25.89" y2="24.13" width="0" layer="19" extent="1-1"/>
+<wire x1="25.89" y1="24.13" x2="22.098" y2="24.13" width="0.381" layer="1"/>
+<wire x1="22.098" y1="24.13" x2="10.94" y2="24.13" width="0.381" layer="1"/>
+<wire x1="22.098" y1="13.462" x2="24.384" y2="13.462" width="0.381" layer="1"/>
+<wire x1="22.098" y1="24.13" x2="22.098" y2="13.462" width="0.381" layer="1"/>
+<wire x1="24.384" y1="13.462" x2="24.511" y2="13.335" width="0.381" layer="1"/>
 </signal>
 <signal name="VCC">
 <contactref element="U$1" pad="12"/>
 <contactref element="C2" pad="1"/>
-<wire x1="24.511" y1="6.985" x2="35.56" y2="11.85" width="0" layer="19" extent="1-1"/>
+<wire x1="31.242" y1="7.366" x2="35.56" y2="11.684" width="0.381" layer="1"/>
+<wire x1="24.638" y1="7.366" x2="31.242" y2="7.366" width="0.381" layer="1"/>
+<wire x1="24.638" y1="7.112" x2="24.638" y2="7.366" width="0.381" layer="1"/>
+<wire x1="35.56" y1="11.684" x2="35.56" y2="11.85" width="0.381" layer="1"/>
+<wire x1="24.638" y1="7.112" x2="24.511" y2="6.985" width="0.381" layer="1"/>
 </signal>
 <signal name="VSS">
@@
 <contactref element="D13" pad="K"/>
 <contactref element="D14" pad="K"/>
-<wire x1="29.99" y1="39.37" x2="29.99" y2="46.99" width="0" layer="19" extent="1-1"/>
-<wire x1="29.99" y1="31.75" x2="29.99" y2="39.37" width="0" layer="19" extent="1-1"/>
-<wire x1="29.99" y1="24.13" x2="29.99" y2="31.75" width="0" layer="19" extent="1-1"/>
-<wire x1="18.2" y1="49.53" x2="29.99" y2="46.99" width="0" layer="19" extent="1-1"/>
-<wire x1="11.049" y1="10.795" x2="29.99" y2="24.13" width="0" layer="19" extent="1-1"/>
+<wire x1="30.48" y1="31.75" x2="30.48" y2="25.908" width="0.381" layer="1"/>
+<wire x1="30.48" y1="25.908" x2="30.48" y2="24.13" width="0.381" layer="1"/>
+<wire x1="30.48" y1="24.13" x2="29.99" y2="24.13" width="0.381" layer="1"/>
+<wire x1="17.78" y1="50.8" x2="17.78" y2="49.53" width="0.381" layer="1"/>
+<wire x1="19.05" y1="52.07" x2="17.78" y2="50.8" width="0.381" layer="1"/>
+<wire x1="30.48" y1="52.07" x2="19.05" y2="52.07" width="0.381" layer="1"/>
+<wire x1="30.48" y1="46.99" x2="30.48" y2="52.07" width="0.381" layer="1"/>
+<wire x1="17.78" y1="49.53" x2="18.2" y2="49.53" width="0.381" layer="1"/>
+<wire x1="30.48" y1="46.99" x2="30.48" y2="39.37" width="0.381" layer="1"/>
+<wire x1="30.48" y1="46.99" x2="29.99" y2="46.99" width="0.381" layer="1"/>
+<wire x1="30.48" y1="39.37" x2="30.48" y2="31.75" width="0.381" layer="1"/>
+<wire x1="30.48" y1="31.75" x2="29.99" y2="31.75" width="0.381" layer="1"/>
+<wire x1="30.48" y1="39.37" x2="29.99" y2="39.37" width="0.381" layer="1"/>
+<wire x1="12.954" y1="10.922" x2="11.176" y2="10.922" width="0.381" layer="1"/>
+<wire x1="27.94" y1="25.908" x2="12.954" y2="10.922" width="0.381" layer="16"/>
+<wire x1="30.48" y1="25.908" x2="27.94" y2="25.908" width="0.381" layer="16"/>
+<wire x1="11.176" y1="10.922" x2="11.049" y2="10.795" width="0.381" layer="1"/>
+<via x="12.954" y="10.922" extent="1-16" drill="0.6096"/>
+<via x="30.48" y="25.908" extent="1-16" drill="0.6096"/>
 </signal>
 </signals>
